File: RP2350B Multi-module controller PCB/multi-module_controller_PCB.kicad_sch (KiCad schematic)
At the start: 87 parts, among them J1 Conn_02x06_Odd_Even, J10 Internal unused GPIO Breakout, J2 Conn_02x26_Odd_Even, J3 Conn_02x26_Odd_Even, J4 SM03B-SRSS-TB, J5 USB_C_Receptacle_USB2.0_14P, J6 USB_C_Receptacle_USB2.0_14P, J7 Module_Bay, J8 USB_A, J9 ADC_Breakout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

Commit message: start preparing PCB schematic for SD card in version 1.1
Parts:
- added J11: Micro_SD_Card_Det1, symbol Connector:Micro_SD_Card_Det1
Other:
- moved on the sheet: C19, J10
Changed lines of the file:
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@@
 	(wire
 		(pts
-			(xy 365.76 212.09) (xy 373.38 212.09)
+			(xy 353.06 203.2) (xy 360.68 203.2)
 		)
 		(stroke
@@
 	(wire
 		(pts
-			(xy 365.76 214.63) (xy 373.38 214.63)
+			(xy 353.06 205.74) (xy 360.68 205.74)
 		)
 		(stroke
@@
 	(wire
 		(pts
-			(xy 344.17 214.63) (xy 353.06 214.63)
+			(xy 331.47 205.74) (xy 340.36 205.74)
 		)
 		(stroke
@@
 	(wire
 		(pts
-			(xy 341.63 212.09) (xy 353.06 212.09)
+			(xy 328.93 203.2) (xy 340.36 203.2)
 		)
 		(stroke
@@
 	(wire
 		(pts
-			(xy 365.76 217.17) (xy 373.38 217.17)
+			(xy 353.06 208.28) (xy 360.68 208.28)
 		)
 		(stroke
@@
 	(wire
 		(pts
-			(xy 344.17 217.17) (xy 353.06 217.17)
+			(xy 331.47 208.28) (xy 340.36 208.28)
 		)
 		(stroke
@@
 	(wire
 		(pts
-			(xy 304.8 114.3) (xy 304.8 116.84)
+			(xy 307.34 67.31) (xy 307.34 69.85)
 		)
 		(stroke
@@
 	(wire
 		(pts
-			(xy 304.8 124.46) (xy 304.8 125.73)
+			(xy 307.34 77.47) (xy 307.34 78.74)
 		)
 		(stroke
@@
 	)
 	(label "GPIO18"
-		(at 373.38 212.09 180)
+		(at 360.68 203.2 180)
 		(effects
 			(font
@@
 	)
 	(label "GPIO21"
-		(at 344.17 217.17 0)
+		(at 331.47 208.28 0)
 		(effects
 			(font
@@
 	)
 	(label "GPIO19"
-		(at 373.38 214.63 180)
+		(at 360.68 205.74 180)
 		(effects
 			(font
@@
 	)
 	(label "GPIO17"
-		(at 344.17 214.63 0)
+		(at 331.47 205.74 0)
 		(effects
 			(font
@@
 	)
 	(label "GPIO20"
-		(at 373.38 217.17 180)
+		(at 360.68 208.28 180)
 		(effects
 			(font
@@
 	(symbol
 		(lib_id "power:+3V3")
-		(at 304.8 114.3 0)
+		(at 307.34 67.31 0)
 		(unit 1)
 		(body_style 1)
@@
 		(dnp no)
 		(property "Reference" "#PWR023"
-			(at 304.8 118.11 0)
+			(at 307.34 71.12 0)
 			(hide yes)
 			(show_name no)
@@
 		)
 		(property "Value" "+3V3"
-			(at 305.181 109.9058 0)
+			(at 307.721 62.9158 0)
 			(show_name no)
 			(do_not_autoplace no)
@@
 		)
 		(property "Footprint" ""
-			(at 304.8 114.3 0)
+			(at 307.34 67.31 0)
 			(hide yes)
 			(show_name no)
@@
 		)
 		(property "Datasheet" ""
-			(at 304.8 114.3 0)
+			(at 307.34 67.31 0)
 			(hide yes)
 			(show_name no)
@@
 		)
 		(property "Description" ""
-			(at 304.8 114.3 0)
+			(at 307.34 67.31 0)
 			(show_name no)
 			(do_not_autoplace no)
@@
 	(symbol
 		(lib_id "Device:C")
-		(at 304.8 120.65 0)
+		(at 307.34 73.66 0)
 		(unit 1)
 		(body_style 1)
@@
 		(dnp no)
 		(property "Reference" "C19"
-			(at 307.721 119.4816 0)
+			(at 310.261 72.4916 0)
 			(show_name no)
 			(do_not_autoplace no)
@@
 		)
 		(property "Value" "10u"
-			(at 307.721 121.793 0)
+			(at 310.261 74.803 0)
 			(show_name no)
 			(do_not_autoplace no)
@@
 		)
 		(property "Footprint" "Capacitor_SMD:C_0805_2012Metric"
-			(at 305.7652 124.46 0)
+			(at 308.3052 77.47 0)
 			(hide yes)
 			(show_name no)
@@
 		)
 		(property "Datasheet" ""
-			(at 304.8 120.65 0)
+			(at 307.34 73.66 0)
 			(hide yes)
 			(show_name no)
@@
 		)
 		(property "Description" ""
-			(at 304.8 120.65 0)
+			(at 307.34 73.66 0)
 			(show_name no)
 			(do_not_autoplace no)
@@
 		)
 		(property "LCSC" "C15850"
-			(at 307.721 119.4816 0)
+			(at 310.261 72.4916 0)
 			(hide yes)
 			(show_name no)
@@
 	(symbol
 		(lib_id "power:GND")
-		(at 304.8 125.73 0)
+		(at 307.34 78.74 0)
 		(unit 1)
 		(body_style 1)
@@
 		(dnp no)
 		(property "Reference" "#PWR024"
-			(at 304.8 132.08 0)
+			(at 307.34 85.09 0)
 			(hide yes)
 			(show_name no)
@@
 		)
 		(property "Value" "GND"
-			(at 300.99 127 0)
+			(at 303.53 80.01 0)
 			(show_name no)
 			(do_not_autoplace no)
@@
 		)
 		(property "Footprint" ""
-			(at 304.8 125.73 0)
+			(at 307.34 78.74 0)
 			(hide yes)
 			(show_name no)
@@
 		)
 		(property "Datasheet" ""
-			(at 304.8 125.73 0)
+			(at 307.34 78.74 0)
 			(hide yes)
 			(show_name no)
@@
 		)
 		(property "Description" ""
-			(at 304.8 125.73 0)
+			(at 307.34 78.74 0)
 			(show_name no)
 			(do_not_autoplace no)
@@
 	(symbol
 		(lib_id "Connector_Generic:Conn_02x03_Odd_Even")
-		(at 358.14 214.63 0)
+		(at 345.44 205.74 0)
 		(unit 1)
 		(body_style 1)
@@
 		(fields_autoplaced yes)
 		(property "Reference" "J10"
-			(at 359.41 206.6755 0)
+			(at 346.71 197.7855 0)
 			(show_name no)
 			(do_not_autoplace no)
@@
 		)
 		(property "Value" "Internal unused GPIO Breakout"
-			(at 359.41 209.0998 0)
+			(at 346.71 200.2098 0)
 			(show_name no)
 			(do_not_autoplace no)
@@
 		)
 		(property "Footprint" "Connector_PinHeader_1.27mm:PinHeader_2x03_P1.27mm_Vertical"
-			(at 358.14 214.63 0)
+			(at 345.44 205.74 0)
 			(hide yes)
 			(show_name no)
@@
 		)
 		(property "Datasheet" ""
-			(at 358.14 214.63 0)
+			(at 345.44 205.74 0)
 			(hide yes)
 			(show_name no)
@@
 		)
 		(property "Description" "Generic connector, double row, 02x03, odd/even pin numbering scheme (row 1 odd numbers, row 2 even numbers), script generated (kicad-library-utils/schlib/autogen/connector/)"
-			(at 358.14 214.63 0)
+			(at 345.44 205.74 0)
 			(hide yes)
 			(show_name no)
@@
 		(lib_name "GND_10")
 		(lib_id "power:GND")
-		(at 341.63 212.09 0)
+		(at 328.93 203.2 0)
 		(unit 1)
 		(body_style 1)
@@
 		(fields_autoplaced yes)
 		(property "Reference" "#PWR055"
-			(at 341.63 218.44 0)
+			(at 328.93 209.55 0)
 			(hide yes)
 			(show_name no)
@@
 		)
 		(property "Value" "GND"
-			(at 341.63 216.2231 0)
+			(at 328.93 207.3331 0)
 			(show_name no)
 			(do_not_autoplace no)
@@
 		)
 		(property "Footprint" ""
-			(at 341.63 212.09 0)
+			(at 328.93 203.2 0)
 			(hide yes)
 			(show_name no)
@@
 		)
 		(property "Datasheet" ""
-			(at 341.63 212.09 0)
+			(at 328.93 203.2 0)
 			(hide yes)
 			(show_name no)
@@
 		)
 		(property "Description" "Power symbol creates a global label with name \"GND\" , ground"
-			(at 341.63 212.09 0)
+			(at 328.93 203.2 0)
 			(hide yes)
 			(show_name no)
@@
 					(unit 1)
 				)
+			)
+		)
+	)
+	(symbol
+		(lib_id "Connector:Micro_SD_Card_Det1")
+		(at 293.37 176.53 0)
+		(unit 1)
+		(body_style 1)
+		(exclude_from_sim no)
+		(in_bom yes)
+		(on_board yes)
+		(in_pos_files yes)
+		(dnp no)
+		(fields_autoplaced yes)
+		(property "Reference" "J11"
+			(at 294.005 154.94 0)
+			(show_name no)
+			(do_not_autoplace no)
+			(effects
+				(font
+					(size 1.27 1.27)
+				)
+			)
+		)
+		(property "Value" "Micro_SD_Card_Det1"
+			(at 294.005 157.48 0)
+			(show_name no)
+			(do_not_autoplace no)
+			(effects
+				(font
+					(size 1.27 1.27)
+				)
+			)
+		)
+		(property "Footprint" ""
+			(at 345.44 158.75 0)
+			(hide yes)
+			(show_name no)
+			(do_not_autoplace no)
+			(effects
+				(font
+					(size 1.27 1.27)
+				)
+			)
+		)
+		(property "Datasheet" "https://datasheet.lcsc.com/lcsc/2110151630_XKB-Connectivity-XKTF-015-N_C381082.pdf"
+			(at 293.37 173.99 0)
+			(hide yes)
+			(show_name no)
+			(do_not_autoplace no)
+			(effects
+				(font
+					(size 1.27 1.27)
+				)
+			)
+		)
+		(property "Description" "Micro SD Card Socket with one card detection pin"
+			(at 293.37 176.53 0)
+			(hide yes)
+			(show_name no)
+			(do_not_autoplace no)
+			(effects
+				(font
+					(size 1.27 1.27)
+				)
+			)
+		)
+		(pin "4"
+		)
+		(pin "3"
+		)
+		(pin "2"
+		)
+		(pin "1"
+		)
+		(pin "SH"
+		)
+		(pin "5"
+		)
+		(pin "6"
+		)
+		(pin "7"
+		)
+		(pin "8"
+		)
+		(pin "9"
+		)
+		(instances
+			(project "multi-module_controller_PCB"
+				(path "/94683f5c-9cd9-448e-be96-9792537b5cb8"
+					(reference "J11")
+					(unit 1)
+				)

Commit message: Add SD Card slot to underside of board, wired for use with SPI1. Reconfigure button pinout and use J10 pins for this purpose
Parts:
- J11: footprint (none) -> EasyEDA:SD-SMD_MLD-TF-PUSH-H18
Connections:
- net +3V3: now also J11.4 (VDD)
- net GND: now also J11.6 (VSS)
- net GPIO17: now also SW9.2; no longer J10.3 (Pin_3)
- net GPIO18: now also SW3.2; no longer J10.2 (Pin_2)
- net GPIO19: now also SW4.2; no longer J10.4 (Pin_4)
- net GPIO20: now also SW5.2; no longer J10.6 (Pin_6)
- net GPIO21: now also SW6.2; no longer J10.5 (Pin_5)
- net GPIO25: now also J11.2 (DAT3/CD); no longer SW9.2
- net GPIO26: now also J11.5 (CLK); no longer SW3.2
- net GPIO27: now also J11.3 (CMD); no longer SW4.2
- net GPIO28: now also J11.7 (DAT0); no longer SW5.2
- net GPIO29: now also J11.CD (DET); no longer SW6.2
- no-connect marks 3 -> 5
Other:
- note added: "REV 2 Changes: Reduce R22, R21, and R20 from 330Ω (or 680Ω) to 22Ω, improving signal response time Add R26 protection resistor Increase R25 from 220Ω to 470Ω to reduce LED brightness Add SD card slot"
- note added: "SPI1 CS"
- note added: "SPI1 MISO"
- note added: "SPI1 MOSI"
- note added: "SPI1 SCK"
- note added: "TODO: shift J10 pins to push buttons to free up GPIO 25-28 or so for SD card SPI1"
- note removed: "REV 2 Changes: Reduce R22, R21, and R20 from 330Ω (or 680Ω) to 22Ω, improving signal response time Add R26 protection resistor Increase R25 from 220Ω to 470Ω to reduce LED brightness"
- moved on the sheet: J10, J11, J4, SW3, SW4, SW5, SW6, SW9

Commit message: Update todo and done details on schematic, start on 3D model for case
Other:
- note added: "REV 2 Changes: Reduce R22, R21, and R20 from 330Ω (or 680Ω) to 22Ω, improving signal response time Add R26 protection resistor Increase R25 from 220Ω to 470Ω to reduce LED brightness Switch VBUS to 3v3 power for display Add SD card slot Reassign pins for UI buttons as required by SD card"
- note added: "REV 2 TODO: Consider always-on power to USB C CC pins - use ADC to detect downstream devices and auto-switch active port Adjust USB traces for proper impedance matching Potentially adjust mounting hole diameter for better compatibility with M3"
- note added: "TODO: remove internal unused GPIO breakout or assign other pins"
- note removed: "REV 2 Changes: Reduce R22, R21, and R20 from 330Ω (or 680Ω) to 22Ω, improving signal response time Add R26 protection resistor Increase R25 from 220Ω to 470Ω to reduce LED brightness Add SD card slot"
- note removed: "REV 2 TODO: Consider always-on power to USB C CC pins - use ADC to detect downstream devices and auto-switch active port"
- note removed: "TODO: shift J10 pins to push buttons to free up GPIO 25-28 or so for SD card SPI1"
Changed lines of the file:
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@@
 		)
 	)
-	(text "REV 2 TODO:\nConsider always-on power to USB C CC pins\n- use ADC to detect downstream devices and auto-switch active port"
-		(exclude_from_sim no)
-		(at 43.942 312.928 0)
+	(text "REV 2 TODO:\nConsider always-on power to USB C CC pins\n- use ADC to detect downstream devices and auto-switch active port\nAdjust USB traces for proper impedance matching\nPotentially adjust mounting hole diameter for better compatibility with M3"
+		(exclude_from_sim no)
+		(at 42.164 319.278 0)
 		(effects
 			(font
@@
 		)
 	)
-	(text "REV 2 Changes:\nReduce R22, R21, and R20 from 330Ω (or 680Ω) to 22Ω, improving signal response time\nAdd R26 protection resistor\nIncrease R25 from 220Ω to 470Ω to reduce LED brightness\nAdd SD card slot"
-		(exclude_from_sim no)
-		(at 40.132 348.996 0)
+	(text "REV 2 Changes:\nReduce R22, R21, and R20 from 330Ω (or 680Ω) to 22Ω, improving signal response time\nAdd R26 protection resistor\nIncrease R25 from 220Ω to 470Ω to reduce LED brightness\nSwitch VBUS to 3v3 power for display\nAdd SD card slot\nReassign pins for UI buttons as required by SD card"
+		(exclude_from_sim no)
+		(at 43.434 376.174 0)
 		(effects
 			(font
@@
 		)
 	)
-	(text "TODO: shift J10 pins to push buttons to\nfree up GPIO 25-28 or so for SD card SPI1"
-		(exclude_from_sim no)
-		(at 367.03 225.298 0)
-		(effects
-			(font
+	(text "TODO: remove internal unused GPIO \nbreakout or assign other pins"
+		(exclude_from_sim no)
+		(at 369.824 222.25 0)
+		(effects
+			(font
