File: RP2350B Multi-module controller PCB/multi-module_controller_PCB.kicad_sch (KiCad schematic)
At the start: 88 parts, among them J1 Conn_02x06_Odd_Even, J10 Internal unused GPIO Breakout, J11 Micro_SD_Card_Det1, J2 Conn_02x26_Odd_Even, J3 Conn_02x26_Odd_Even, J4 SM03B-SRSS-TB, J5 USB_C_Receptacle_USB2.0_14P, J6 USB_C_Receptacle_USB2.0_14P, J7 Module_Bay, J8 USB_A, J9 ADC_Breakout, SW1 SW_Push, SW10 BTN_MDL, SW2 SW_Push, SW3 BTN_LEFT, SW4 BTN_UP, SW5 BTN_OK, SW6 BTN_DOWN, SW7 BTN_RIGHT, SW8 BTN_BACK, SW9 BTN_SYS, U1 RP2350_80QFN, U2 NCP1117-3.3_SOT223, U3 W25Q128JVS, U4 DNF, U5 FSUSB42MUX, U6 MIC2026-1xM, Y1 ABM8-272-T3

Commit message: Finalized V2 schematic and PCB
Parts:
- added J12: Conn_01x01, Connector_PinHeader_2.54mm:PinHeader_1x01_P2.54mm_Vertical, symbol Connector_Generic:Conn_01x01
- added R27: 10k, Resistor_SMD:R_0402_1005Metric, symbol Device:R_Small
- added R28: 100k, Resistor_SMD:R_0402_1005Metric, symbol Device:R_Small
- C25: value 0.1u -> 100n
- H1, H2, H3, H4: footprint MountingHole:MountingHole_2.7mm_M2.5 -> MountingHole:MountingHole_3.2mm_M3
Connections:
- net +3V3: now also J10.5 (Pin_5), J10.6 (Pin_6)
- net GND: now also J10.2 (Pin_2), R27.2
- net GPIO47_ADC7: now also R27.1, R28.2
- new net +BATT: J12.1 (Pin_1), R28.1
Other:
- note added: "REV 2 Changes: Reduce R22, R21, and R20 from 330Ω (or 680Ω) to 22Ω, improving signal response time Add R26 protection resistor Increase R25 from 220Ω to 470Ω to reduce LED brightness Switch VBUS to 3v3 power for display Add SD card slot Reassign pins for UI buttons as required by SD card Add Battery-sense input to GPIO47 (ADC7)"
- note removed: "REV 2 Changes: Reduce R22, R21, and R20 from 330Ω (or 680Ω) to 22Ω, improving signal response time Add R26 protection resistor Increase R25 from 220Ω to 470Ω to reduce LED brightness Switch VBUS to 3v3 power for display Add SD card slot Reassign pins for UI buttons as required by SD card"
- moved on the sheet: J10
