File: RP2350B Multi-module controller PCB/multi-module_controller_PCB.kicad_pcb (KiCad board)
At the start: 4 copper layers, 59.8 x 84.4 mm, 86 parts, among them J1 Conn_02x06_Odd_Even, J10 Internal unused GPIO Breakout, J11 Micro_SD_Card_Det1, J4 SM03B-SRSS-TB, J5 USB_C_Receptacle_USB2.0_14P, J6 USB_C_Receptacle_USB2.0_14P, J7 Module_Bay, J8 USB_A, J9 ADC_Breakout, SW1 SW_Push, SW10 BTN_MDL, SW2 SW_Push, SW3 BTN_LEFT, SW4 BTN_UP, SW5 BTN_OK, SW6 BTN_DOWN, SW7 BTN_RIGHT, SW8 BTN_BACK, SW9 BTN_SYS, U1 RP2350_80QFN, U2 NCP1117-3.3_SOT223, U3 W25Q128JVS, U4 DNF, U5 FSUSB42MUX, U6 MIC2026-1xM, Y1 ABM8-272-T3

Commit message: Finalized V2 schematic and PCB
Parts:
- added J12: Conn_01x01, Connector_PinHeader_2.54mm:PinHeader_1x01_P2.54mm_Vertical, F.Cu at (73.9, 76.7)
- added R27: 10k, Resistor_SMD:R_0402_1005Metric, F.Cu at (74.2, 82.5)
- added R28: 100k, Resistor_SMD:R_0402_1005Metric, F.Cu at (71.2, 82.5)
- C25: value 0.1u -> 100n
- H1, H2, H3, H4: footprint MountingHole:MountingHole_2.7mm_M2.5 -> MountingHole:MountingHole_3.2mm_M3
- J4: value SM03B-SRSS-TB -> Conn_Generic 1x3
Connections:
- J10 pad 2: unconnected-(J10-Pin_2-Pad2) -> GND
- J10 pad 5: unconnected-(J10-Pin_5-Pad5) -> +3V3
- J10 pad 6: unconnected-(J10-Pin_6-Pad6) -> +3V3
Routing:
- net /GPIO47_ADC7: track 12.8 -> 88.9 mm
- net +BATT: track 0.00 -> 7.14 mm
- net GND: track 162.7 -> 167.7 mm
- net /GPIO29: track 39.9 -> 35.3 mm
- net /GPIO30: track 35.4 -> 32.9 mm, vias 2 -> 0
Other:
- board text added: "2.0"
- board text added: "V2.0 2025-2026"
- board text added: "VBAT"
- board text removed: "1.1"
- board text removed: "V1.1 2025-2026"
